File: kicad/fli3dv2.kicad_pcb (KiCad board)
At the start: 2 copper layers, 35 x 138 mm, 20 parts, among them J1 BAT connector, J2 Conn_Serial, J3 Separation Detect, J4 Parachute Release, J5 Conn_Power, J7 Conn_IO, K1 HFD4_4.5-SR, SW1 PWR jumper, SW2 SW_DIP, U3 ESP32-CAM, U8 esp32-wemos-d1-mini

Commit message: PCB v0.4.1: set GY912 on 3.3V and decoupled ESP32CAM GND/R
Connections:
- SW2 pad 3: 5V PWR -> 3.3V PWR
- U3 pad 9: GND -> unconnected-(U3-GND-Pad9)
Routing:
- net 3.3V PWR: track 40.8 -> 42.1 mm
- net 5V PWR: track 32.9 -> 31.7 mm
Other:
- board text added: "Fli3d v2 PCB 0.4.1 (front)"
- board text added: "Fli3d v2 PCB 0.4.1 (rear)"
- board text removed: "Fli3d v2 PCB 0.4.0 (front)"
- board text removed: "Fli3d v2 PCB 0.4.0 (rear)"
